File: esp_garden_v2.brd (EAGLE design)
At the start: 50 x 100 mm, 33 parts, among them T1 DMN6068SE-13, T2 DMN6068SE-13, T3 DMN6068SE-13, T4 DMN6068SE-13, U1 V1, U10 V1, U11 V1, U12 V1, U14 V1, U15 V1, U2 V1, U3 V1, U4 V1, U6 V1

Commit message: Ordered version
Parts:
- moved R2 63.0 mm to (39.5, 23.0), turned to 270 degrees
- moved R4 63.0 mm to (39.5, 17.0), turned to 270 degrees
- moved R5 57.2 mm to (37.5, 19.0), turned to 90 degrees
- moved R1 32.0 mm to (39.5, 50.5), turned to 90 degrees
Routing:
- net N$2: track 24.4 -> 38.1 mm, vias 1 -> 2
- net SDA/DHT: track 98.8 -> 103.8 mm
- net TEMP: track 44.4 -> 49.0 mm
- net RELAY_0: track 95.9 -> 96.8 mm
- net +3V3: track 58.1 -> 57.5 mm, vias 2 -> 1
Other:
- board text removed: "+12V"
